File: puzzlekeyboard/puzzlekeyboard.kicad_sch (KiCad schematic)
At the start: 16 parts, among them J1 Conn_01x01_Pin, J10 Conn_01x01_Socket, J11 Conn_01x05_Socket, J12 Conn_01x05_Socket, J2 Conn_01x01_Pin, J3 Conn_01x01_Socket, J4 Conn_01x01_Socket, J5 Conn_01x05_Socket, J6 Conn_01x05_Pin, J7 Conn_01x01_Socket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

Commit message: a
Parts:
- added J13, J15: Conn_01x01_Socket, symbol Connector:Conn_01x01_Socket
- added J14, J16: Conn_01x01_Pin, symbol Connector:Conn_01x01_Pin
- added SW2: SW_SPST, symbol Switch:SW_SPST
Connections:
- net IO: now reaches U1.11 (P1.15_D10_MOSI)
- net IO: now also SW2.1 (A)
- net GND: now reaches U1.13 (GND)
- net GND: now also SW2.2 (B)
- new net: J14.1 (Pin_1), J15.1 (Pin_1)
- new net: J13.1 (Pin_1), J16.1 (Pin_1)
- no-connect marks 2 -> 4
Other:
- note added: "IO_switch"
- note added: "Voidkey_unit"

Commit message: a
a
Parts:
- removed J5, J9: Conn_01x05_Socket, symbol Connector:Conn_01x05_Socket
- added J17, J18: Conn_01x04_Socket, symbol Connector:Conn_01x04_Socket
Connections:
- net at J6.2 (Pin_2): now also J18.1 (Pin_1)
- net at J6.3 (Pin_3): now also J18.2 (Pin_2)
- net at J6.4 (Pin_4): now also J18.3 (Pin_3)
- net at J6.5 (Pin_5): now also J18.4 (Pin_4)
- net at J8.1 (Pin_1): now also J17.1 (Pin_1)
- net at J8.2 (Pin_2): now also J17.2 (Pin_2)
- net at J8.3 (Pin_3): now also J17.3 (Pin_3)
- net at J8.4 (Pin_4): now also J17.4 (Pin_4)
- no-connect marks 4 -> 2
Other:
- moved on the sheet: J12, U1
